File: tests/projects/basic/basic.kicad_sch (KiCad schematic)
At the start: 4 parts

Commit message: fix: honor KiCad DNP symbol flags
Parts:
- added R4: 1k, symbol Device:R
Changed lines of the file:
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@@
     (property "Reference" "R3")
     (property "Value" "1k")
-    (property "DNP" "yes")))
+    (property "DNP" "yes"))
+  (symbol (lib_id "Device:R") (in_bom yes) (dnp yes)
+    (property "Reference" "R4")
+    (property "Value" "1k")))
