File: tests/fixtures/board_minimal.kicad_pcb (KiCad board)
At the start: 2 copper layers, 40 x 10 mm, 0 parts

Commit message: feat: extract assembly placement metrics
Parts:
- added J1: , Connector_THT:USB_B, B.Cu at (0.00, 0.00)
- added R1: , Resistor_SMD:R_0603_1608Metric, F.Cu at (0.00, 0.00)
Changed lines of the file:
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@@
   (gr_line (start 50 20) (end 50 30) (layer "Edge.Cuts"))
   (gr_line (start 50 30) (end 10 30) (layer "Edge.Cuts"))
-  (gr_line (start 10 30) (end 10 20) (layer "Edge.Cuts")))
+  (gr_line (start 10 30) (end 10 20) (layer "Edge.Cuts"))
+  (footprint "Resistor_SMD:R_0603_1608Metric"
+    (layer "F.Cu")
+    (property "Reference" "R1")
+    (attr smd))
+  (footprint "Connector_THT:USB_B"
+    (layer "B.Cu")
+    (property "Reference" "J1")
+    (attr through_hole)))

Commit message: feat: check assembly package capabilities
Parts:
- added U1: , Package_BGA:BGA-4_2x2_0.5mm, F.Cu at (0.00, 0.00)
Changed lines of the file:
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@@
     (layer "B.Cu")
     (property "Reference" "J1")
-    (attr through_hole)))
+    (attr through_hole))
+  (footprint "Package_BGA:BGA-4_2x2_0.5mm"
+    (layer "F.Cu")
+    (property "Reference" "U1")
+    (attr smd)
+    (pad "1" smd circle (at 0 0) (size 0.25 0.25))
+    (pad "2" smd circle (at 0.5 0) (size 0.25 0.25))
+    (pad "3" smd circle (at 0 0.5) (size 0.25 0.25))
+    (pad "4" smd circle (at 0.5 0.5) (size 0.25 0.25))))
